File: pcb-s16/pcb.kicad_pcb (KiCad board)
At the start: 2 copper layers, 28.8 x 14 mm, 12 parts, among them J1 USB_B_Micro, SW1 BTN, U1 PFS154-S16, U2 74HC595, U3 SLR0394DRC5BD, Y1 32.768kHz

Commit message: Update Crystal
Parts:
- Y1: footprint Crystal:Crystal_DS26_D2.0mm_L6.0mm_Horizontal -> Crystal:Crystal_C26-LF_D2.1mm_L6.5mm_Horizontal
Connections:
- net /R3 renamed /e
- net /R4 renamed /f
- net /R7 renamed /g
- net /R8 renamed /dp

Commit message: Add values (680 ohm) for resistor arrays
Parts:
- RN1, RN2: value R_Pack04 -> 680
Changed lines of the file:
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@@
       (effects (font (size 0.6 0.6) (thickness 0.08)))
     )
-    (fp_text value R_Pack04 (at 0 2.8 90) (layer F.Fab)
+    (fp_text value 680 (at 0 2.8 90) (layer F.Fab)
       (effects (font (size 1 1) (thickness 0.15)))
     )
@@
       (effects (font (size 0.6 0.6) (thickness 0.08)))
     )
-    (fp_text value R_Pack04 (at 0 2.8 90) (layer F.Fab) hide
+    (fp_text value 680 (at 0 2.8 90) (layer F.Fab) hide
       (effects (font (size 1 1) (thickness 0.15)))
     )
